File: 04 - POE FONTE EXT- SEM LED/POE FONTE EXT- SEM LED/POE FONTE EXT- SEM LED.kicad_pcb (KiCad board)
At the start: 2 copper layers, 76.8 x 50.8 mm, 7 parts, among them J1 RJ45-8P8C, J2 RJ45-8P8C, J3 DCJ200-10-A-XX-K_REVA

Commit message: Subindo Projeto POE
Parts:
- moved J3 19.3 mm to (128.5, 65.6)
Routing:
- net GND: track 88.6 -> 91.9 mm
- net Net-(F1-Pad1): track 14.1 -> 11.4 mm
Other:
- board size 76.8 x 50.8 mm -> 60 x 50.6 mm
Changed lines of the file:
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@@
 	(footprint "Equatorial_foot:GCT_DCJ200-10-A-XX-K_REVA"
 		(layer "F.Cu")
-		(at 145.1 75.475 90)
+		(at 128.5 65.575 90)
 		(property "Reference" "J3"
-			(at 9.4 -1.8 180)
+			(at 3.5 -11.075 180)
 			(layer "F.SilkS")
 			(effects
@@
 	)
 	(gr_rect
-		(start 75.775 58.3)
-		(end 152.55 109.05)
+		(start 75.775 58.35)
+		(end 135.825 109)
 		(stroke
 			(width 0.05)
@@
 	(gr_rect
 		(start 75.775 58.35)
-		(end 152.5 109)
+		(end 135.825 109)
 		(stroke
 			(width 0.1)
@@
 		)
 	)
-	(segment
-		(start 138.5 75.925)
-		(end 138.55 75.875)
-		(width 1.5)
-		(layer "F.Cu")
-		(net 1)
-	)
-	(segment
-		(start 138.55 75.875)
-		(end 138.55 75.475)
-		(width 1.5)
-		(layer "F.Cu")
-		(net 1)
-	)
-	(segment
-		(start 138.55 75.475)
-		(end 138.425 75.6)
+	(dimension
+		(type aligned)
+		(layer "F.Cu")
+		(pts
+			(xy 75.775 58.35) (xy 135.825 58.35)
+		)
+		(height -6.15)
+		(gr_text "60,0500 mm"
+			(at 105.8 50.4 0)
+			(layer "F.Cu")
+			(effects
+				(font
+					(size 1.5 1.5)
+					(thickness 0.3)
+				)
+			)
+		)
+		(format
+			(prefix "")
+			(suffix "")
+			(units 3)
+			(units_format 1)
+			(precision 4)
+		)
+		(style
+			(thickness 0.2)
+			(arrow_length 1.27)
+			(text_position_mode 0)
+			(extension_height 0.58642)
+			(extension_offset 0.5) keep_text_aligned)
+	)
+	(dimension
+		(type aligned)
+		(layer "F.Cu")
+		(pts
+			(xy 135.825 109) (xy 135.825 58.35)
+		)
+		(height 5.45)
+		(gr_text "50,6500 mm"
+			(at 139.475 83.675 90)
+			(layer "F.Cu")
+			(effects
+				(font
+					(size 1.5 1.5)
+					(thickness 0.3)
+				)
+			)
+		)
+		(format
+			(prefix "")
+			(suffix "")
+			(units 3)
+			(units_format 1)
+			(precision 4)
+		)
+		(style
+			(thickness 0.2)
+			(arrow_length 1.27)
+			(text_position_mode 0)
+			(extension_height 0.58642)
+			(extension_offset 0.5) keep_text_aligned)
+	)
+	(segment
+		(start 121.95 67.4)
+		(end 125.05 70.5)
 		(width 1.5)
 		(layer "F.Cu")
@@
 	)
 	(segment
-		(start 138.425 75.6)
+		(start 125.05 70.5)
 		(end 125.05 75.6)
+		(width 1.5)
+		(layer "F.Cu")
+		(net 1)
+	)
+	(segment
+		(start 121.95 65.575)
+		(end 121.95 67.4)
 		(width 1.5)
 		(layer "F.Cu")
@@
 	)
 	(segment
-		(start 133.275 106.025)
-		(end 144.85 94.45)
-		(width 1)
+		(start 124.85 62.175)
+		(end 124.85 60.775)
+		(width 2)
 		(layer "F.Cu")
 		(net 4)
@@
 	)
 	(segment
-		(start 144.85 94.45)
-		(end 144.85 75.475)
-		(width 1)
-		(layer "F.Cu")
-		(net 4)
-	)
-	(segment
-		(start 144.85 74.075)
-		(end 141.45 70.675)
-		(width 2)
-		(layer "F.Cu")
-		(net 4)
-	)
-	(segment
 		(start 110.45 106.025)
 		(end 106.55 106.025)
@@
 	)
 	(segment
+		(start 124.85 60.775)
+		(end 124.75 60.875)
+		(width 2)
+		(layer "F.Cu")
+		(net 4)
+	)
+	(segment
+		(start 128.25 67.4)
+		(end 132.15 71.3)
+		(width 1.2)
+		(layer "F.Cu")
+		(net 4)
+	)
+	(segment
 		(start 103.475 102.95)
 		(end 106.55 106.025)
@@
 	)
 	(segment
+		(start 131.025 106.025)
+		(end 110.45 106.025)
+		(width 1.2)
+		(layer "F.Cu")
+		(net 4)
+	)
+	(segment
 		(start 110.325 106.15)
 		(end 110.45 106.025)
@@
 	)
 	(segment
-		(start 144.85 75.475)
-		(end 144.85 74.075)
-		(width 1)
+		(start 132.15 71.3)
+		(end 132.15 104.9)
+		(width 1.2)
+		(layer "F.Cu")
+		(net 4)
+	)
+	(segment
+		(start 132.15 104.9)
+		(end 131.025 106.025)
+		(width 1.2)
 		(layer "F.Cu")
 		(net 4)
@@
 	)
 	(segment
-		(start 110.45 106.025)
-		(end 133.275 106.025)
-		(width 1)
+		(start 128.25 65.575)
+		(end 124.85 62.175)
+		(width 2)
 		(layer "F.Cu")
 		(net 4)
